Commit message: added moveit

File: hannahbot_description/urdf/hannahbot.urdf.xacro (robot description, xacro)
@@ -1,241 +1,182 @@
 <?xml version="1.0"?>
-<robot xmlns:xacro="http://www.ros.org/wiki/xacro" name="hannah_bot">
-  <xacro:include filename="$(find hannahbot_description)/urdf/hannahbot_gazebo.xacro"/>
-  <xacro:include filename="$(find hannahbot_description)/urdf/hannahbot_ros2_control.xacro"/>
-  <xacro:property name="PI" value="3.14159"/>
-  <xacro:property name="effort" value="30.0"/>
-  <xacro:property name="velocity" value="10.0"/>
-  <xacro:macro name="default_inertial" params="mass">
-    <inertial>
-      <mass value="${mass}"/>
-      <inertia ixx="1.0" ixy="0.0" ixz="0.0"
-                iyy="1.0" iyz="0.0"
-                izz="1.0" />
-    </inertial>
-  </xacro:macro>
-  <xacro:macro name="default_transmission" params="number" >
-    <transmission name="transmission_${number}">
-      <plugin>transmission_interfaces/SimpleTransmission</plugin>
-      <actuator name="motor_${number}" role="actuator1"/>
-      <joint name="joint_${number}" role="joint1">
-        <mechanical_reduction>1.0</mechanical_reduction>
-      </joint>
-    </transmission>
-  </xacro:macro>
-  <link name="world"/>
-  <xacro:default_inertial mass="1.0"/>
-  <link name="base_link">
-    <visual>
-    <origin rpy="0 0 0" xyz="-0.5 -0.5 0"/>
-      <geometry>
-        <mesh filename="package://hannahbot_description/meshes/basement.STL" scale="0.01 0.01 0.01"/>
-      </geometry>
-    </visual>
-    <collision>
-      <origin rpy="0 0 0" xyz="-0.5 -0.5 0"/>
-      <geometry>
-        <mesh filename="package://hannahbot_description/meshes/basement.STL" scale="0.01 0.01 0.01"/>
-      </geometry>
-    </collision>
+<robot xmlns:xacro="http://www.ros.org/wiki/xacro" name="hannahbot">
+    <!-- Start GZ or Ignition depending on ROS 2 Version -->
+    <xacro:arg name="is_ignition" default="true"/>
+    <!-- Include Gazebo Parameters -->
+    <xacro:include filename="$(find hannahbot_description)/urdf/hannahbot_gazebo.xacro" />
+    <!-- Include ros2_control Plugins -->
+    <xacro:include filename="$(find hannahbot_description)/urdf/hannahbot_ros2_control.xacro" />
+    <!-- Useful XACRO Variables (Properties) -->
+    <xacro:property name="PI" value="3.14159265359" />
+    <xacro:property name="effort" value="30.0" />
+    <xacro:property name="velocity" value="10.0" />
+    <!-- Useful Macros -->
+    <xacro:macro name="default_inertial" params="mass">
+        <inertial>
+            <origin xyz="0 0 0" rpy="0 0 0"/>
+            <mass value="${mass}" />
+            <inertia ixx="1.0" ixy="0.0" ixz="0.0"
+                     iyy="1.0" iyz="0.0"
+                     izz="1.0" />
+        </inertial>
+    </xacro:macro>
+    <!-- Links -->
+    <link name="world"/>
+    <link name="base_link">
+        <xacro:default_inertial mass="1.0"/>
+        <visual>
+            <origin rpy="0 0 0" xyz="-0.5 -0.5 0"/>
+            <geometry>
+                <mesh filename="package://hannahbot_description/meshes/basement.STL" scale="0.01 0.01 0.01"/>
+            </geometry>
+        </visual>
+        <collision>
+            <origin rpy="0 0 0" xyz="-0.5 -0.5 0"/>
+            <geometry>
+                <mesh filename="package://hannahbot_description/meshes/basement.STL" scale="0.01 0.01 0.01"/>
+            </geometry>
+        </collision>
     </link>
-    <joint name="please_jesus" type="fixed">
+    <link name="base_plate">
+        <xacro:default_inertial mass="0.1"/>
+        <visual>
+            <origin rpy="0 0 0" xyz="-0.39 -0.39 -0.56"/>
+            <geometry>
+                <mesh filename="package://hannahbot_description/meshes/base_plate.STL" scale="0.01 0.01 0.01"/>
+            </geometry>
+        </visual>
+        <collision>
+            <origin rpy="0 0 0" xyz="-0.39 -0.39 -0.56"/>
+            <geometry>
+                <mesh filename="package://hannahbot_description/meshes/base_plate.STL" scale="0.01 0.01 0.01"/>
+            </geometry>
+        </collision>
+    </link>
+    <link name="forward_drive_arm">
+        <xacro:default_inertial mass="0.1"/>
+        <visual>
+            <origin rpy=" 0 -${PI / 2} ${PI / 2}" xyz="0.19 0.06 -0.08"/>
+            <geometry>
+                <mesh filename="package://hannahbot_description/meshes/forward_drive_arm.STL" scale="0.01 0.01 0.01"/>
+            </geometry>
+        </visual>
+        <collision>
+            <origin rpy=" 0 -${PI / 2} ${PI / 2}" xyz="0.19 0.06 -0.08"/>
+            <geometry>
+                <mesh filename="package://hannahbot_description/meshes/forward_drive_arm.STL" scale="0.01 0.01 0.01"/>
+            </geometry>
+        </collision>
+    </link>
+    <link name="horizontal_arm">
+        <xacro:default_inertial mass="0.1"/>
+        <visual>
+            <origin rpy="${PI / 2} 0 ${PI / 2}" xyz="-0.03 -0.4 -0.06"/>
+            <geometry>
+                <mesh filename="package://hannahbot_description/meshes/horizontal_arm.STL" scale="0.01 0.01 0.01"/>
+            </geometry>
+        </visual>
+        <collision>
+            <origin rpy="${PI / 2} 0 ${PI / 2}" xyz="-0.03 -0.4 -0.06"/>
+            <geometry>
+                <mesh filename="package://hannahbot_description/meshes/horizontal_arm.STL" scale="0.01 0.01 0.01"/>
+            </geometry>
+        </collision>
+    </link>
+    <link name="claw_support">
+        <xacro:default_inertial mass="0.05"/>
+        <visual>
+            <origin rpy="0 0 ${PI / 2}" xyz="0 -0.05 -0.15"/>
+            <geometry>
+                <mesh filename="package://hannahbot_description/meshes/claw_support.STL" scale="0.01 0.01 0.01"/>
+            </geometry>
+        </visual>
+        <collision>
+            <origin rpy="0 0 ${PI / 2}" xyz="0 -0.05 -0.15"/>
+            <geometry>
+                <mesh filename="package://hannahbot_description/meshes/claw_support.STL" scale="0.01 0.01 0.01"/>
+            </geometry>
+        </collision>
+    </link>
+    <link name="gripper_right">
+        <xacro:default_inertial mass="0.01"/>
+        <visual>
+            <origin rpy="0 0 -${PI / 2}" xyz="-0.1 0.50 -0.1"/>
+            <geometry>
+                <mesh filename="package://hannahbot_description/meshes/right_finger.STL" scale="0.01 0.01 0.01"/>
+            </geometry>
+        </visual>
+        <collision>
+            <origin rpy="0 0 -${PI / 2}" xyz="-0.1 0.50 -0.1"/>
+            <geometry>
+                <mesh filename="package://hannahbot_description/meshes/right_finger.STL" scale="0.01 0.01 0.01"/>
+            </geometry>
+        </collision>
+    </link>
+    <link name="gripper_left">
+        <xacro:default_inertial mass="0.01"/>
+        <visual>
+            <origin rpy="0 0 -${PI / 2}" xyz="-0.04 0.50 -0.1"/>
+            <geometry>
+                <mesh filename="package://hannahbot_description/meshes/left_finger.STL" scale="0.01 0.01 0.01"/>
+            </geometry>
+        </visual>
+        <collision>
+            <origin rpy="0 0 -${PI / 2}" xyz="-0.04 0.50 -0.1"/>
+            <geometry>
+                <mesh filename="package://hannahbot_description/meshes/left_finger.STL" scale="0.01 0.01 0.01"/>
+            </geometry>
+        </collision>
+    </link>
+    <!-- Joints -->
+    <joint name="virtual_joint" type="fixed">
         <parent link="world"/>
         <child link="base_link"/>
-        <origin rpy="0 0 0" xyz="0 0 0"/>
+        <origin xyz="0 0 0" rpy="0 0 0"/>
     </joint>
-    <link name="base_plate">
-      <xacro:default_inertial mass="0.1"/>
-      <visual>
-        <origin rpy="0 0 0" xyz="-0.39 -0.39 -0.56"/>
-        <geometry>
-          <mesh filename="package://hannahbot_description/meshes/base_plate.STL" scale="0.01 0.01 0.01"/>
-        </geometry>
-      </visual>
-      <collision>
-          <origin rpy="0 0 0" xyz="-0.39 -0.39 -0.56"/>
-          <geometry>
-            <mesh filename="package://hannahbot_description/meshes/base_plate.STL" scale="0.01 0.01 0.01"/>
-          </geometry>
-      </collision>
-    </link>
-    <joint name="joint_1" type="revolute">
-      <parent link="base_link"/>
-      <child link="base_plate"/>
-      <axis xyz="0 0 1"/>
-      <origin rpy="0 0 0" xyz="0 0 0.307"/>
-      <limit lower="-${PI/2}" upper="${PI/2}" effort="${effort}" velocity="${velocity}"/>
+    <joint name ="joint_1" type="revolute">
+        <parent link="base_link"/>
+        <child link = "base_plate"/>
+        <origin xyz="0 0 0.307"/>
+        <axis xyz="0 0 1"/>
+        <limit lower="-${PI / 2}" upper="${PI / 2}"
+               effort="${effort}" velocity="${velocity}"/>
     </joint>
-    <!-- forward arm -->
-    <link name="forward_drive_link">
-      <xacro:default_inertial mass="0.1"/>
-      <visual>
-        <origin rpy="0 -${PI/2} ${PI/2}" xyz="0.19 0.06 -0.08"/>
-        <geometry>
-          <mesh filename="package://hannahbot_description/meshes/forward_drive_arm.STL" scale="0.01 0.01 0.01"/>
-        </geometry>
-      </visual>
-      <collision>
-        <origin rpy="0 -${PI/2} ${PI/2}" xyz="0.19 0.06 -0.08"/>
-        <geometry>
-          <mesh filename="package://hannahbot_description/meshes/forward_drive_arm.STL" scale="0.01 0.01 0.01"/>
-        </geometry>
-      </collision>
-    </link>
-    <joint name="joint_2" type="revolute">
-      <parent link="base_plate"/>
-      <child link="forward_drive_link"/>
-      <axis xyz="1 0 0"/>
-      <origin rpy="0 0 0" xyz="-0.02 0 0.35"/>
-      <limit lower="-${PI/2}" upper="${PI/2}" effort="${effort}" velocity="${velocity}"/>
+    <joint name ="joint_2" type="revolute">
+        <parent link="base_plate"/>
+        <child link = "forward_drive_arm"/>
+        <origin xyz="-0.02 0 0.35"/>
+        <axis xyz="1 0 0"/>
+        <limit lower="-${PI / 2}" upper="${PI / 2}"
+                effort="${effort}" velocity="${velocity}"/>
     </joint>
-    <!-- horizantal arm -->
-    <link name="horizontal_arm_link">
-      <xacro:default_inertial mass="0.1"/>
-      <visual>
-        <origin rpy="${PI/2} 0 ${PI/2}" xyz="-0.03 -0.4 -0.06"/>
-        <geometry>
-          <mesh filename="package://hannahbot_description/meshes/horizontal_arm.STL" scale="0.01 0.01 0.01"/>
-        </geometry>
-      </visual>
-      <collision>
-        <origin rpy="${PI/2} 0 ${PI/2}" xyz="-0.03 -0.4 -0.06"/>
-        <geometry>
-          <mesh filename="package://hannahbot_description/meshes/horizontal_arm.STL" scale="0.01 0.01 0.01"/>
-        </geometry>
-      </collision>
-    </link>
-    <joint name="joint_3" type="revolute">
-      <parent link="forward_drive_link"/>
-      <child link="horizontal_arm_link"/>
-      <axis xyz="1 0 0"/>
-      <origin rpy="0 0 0" xyz="0 0 0.8"/>
-      <limit lower="-${PI/2}" upper="${PI/2}" effort="${effort}" velocity="${velocity}"/>
+    <joint name ="joint_3" type="revolute">
+        <parent link="forward_drive_arm"/>
+        <child link = "horizontal_arm"/>
+        <origin xyz="0 0 0.8"/>
+        <axis xyz="1 0 0"/>
+        <limit lower="-${PI / 2}" upper="${PI / 2}"
+               effort="${effort}" velocity="${velocity}"/>
     </joint>
-    <!-- claw  -->
-    <link name="claw_support">
-      <xacro:default_inertial mass="0.05"/>
-      <visual>
-        <origin rpy="0 0 ${PI/2}" xyz="0 -0.05 -0.15"/>
-        <geometry>
-          <mesh filename="package://hannahbot_description/meshes/claw_support.STL" scale="0.01 0.01 0.01"/>
-        </geometry>
-      </visual>
-      <collision>
-        <origin rpy="0 0 ${PI/2}" xyz="0 -0.05 -0.15"/>
-        <geometry>
-          <mesh filename="package://hannahbot_description/meshes/claw_support.STL" scale="0.01 0.01 0.01"/>
-        </geometry>
-      </collision>
-    </link>
-    <joint name="hori_arm_claw_joint" type="revolute">
-      <parent link="horizontal_arm_link"/>
-      <child link="claw_support"/>
-      <axis xyz="1 0 0"/>
-      <origin rpy="0 0 0" xyz="0 0.82 0"/>
-      <limit lower="-${PI/2}" upper="${PI/2}" effort="${effort}" velocity="${velocity}"/>
+    <joint name ="horizontal_arm_to_claw_support" type="fixed">
+        <parent link="horizontal_arm"/>
+        <child link = "claw_support"/>
+        <origin xyz="0 0.82 0"/>
     </joint>
-     <!-- gripper_right -->
-     <link name="gripper_right">
-      <xacro:default_inertial mass="0.01"/>
-      <visual>
-        <origin rpy="0 0 -${PI/2}" xyz="-0.1 0.5 -0.1"/>
-        <geometry>
-          <mesh filename="package://hannahbot_description/meshes/right_finger.STL" scale="0.01 0.01 0.01"/>
-        </geometry>
-      </visual>
-      <collision>
-        <origin rpy="0 0 -${PI/2}" xyz="-0.1 0.5 -0.1"/>
-        <geometry>
-          <mesh filename="package://hannahbot_description/meshes/right_finger.STL" scale="0.01 0.01 0.01"/>
-        </geometry>
-      </collision>
-    </link>
-    <joint name="joint_4" type="revolute">
-      <parent link="claw_support"/>
-      <child link="gripper_right"/>
-      <axis xyz="0 0 1"/>
-      <origin rpy="0 0 0" xyz="-0.04 0.13 -0.1"/>
-      <limit lower="-${PI/2}" upper="0.0" effort="${effort}" velocity="${velocity}"/>
+    <joint name ="joint_4" type="revolute">
+        <parent link="claw_support"/>
+        <child link = "gripper_right"/>
+        <origin xyz="-0.04 0.13 -0.1"/>
+        <axis xyz="0 0 1"/>
+        <limit lower="-${PI / 2}" upper="0.0"
+               effort="${effort}" velocity="${velocity}"/>
     </joint>
-      <!-- gripper_left -->
-      <link name="gripper_left">
-        <xacro:default_inertial mass="0.01"/>
-        <visual>
-          <origin rpy="0 0 -${PI/2}" xyz="-0.04 0.5 -0.1"/>
-          <geometry>
-            <mesh filename="package://hannahbot_description/meshes/left_finger.STL" scale="0.01 0.01 0.01"/>
-          </geometry>
-        </visual>
-        <collision>
-          <origin rpy="0 0 -${PI/2}" xyz="-0.04 0.5 -0.1"/>
-          <geometry>
-            <mesh filename="package://hannahbot_description/meshes/left_finger.STL" scale="0.01 0.01 0.01"/>
-          </geometry>
-        </collision>
-      </link>
-      <joint name="joint_5" type="revolute">
+    <joint name ="joint_5" type="revolute">
         <parent link="claw_support"/>
-        <child link="gripper_left"/>
+        <child link = "gripper_left"/>
+        <origin xyz="-0.22 0.13 -0.1"/>
         <axis xyz="0 0 1"/>
-        <origin rpy="0 0 0" xyz="-0.22 0.13 -0.1"/>
+        <limit lower="0.0" upper="${PI / 2}"
+               effort="${effort}" velocity="${velocity}"/>
         <mimic joint="joint_4" multiplier="-1"/>
-        <limit lower="0.0" upper="${PI/2}" effort="${effort}" velocity="${velocity}"/>
-      </joint>
-      <xacro:default_transmission number="1"/>
-      <xacro:default_transmission number="2"/>
-      <xacro:default_transmission number="3"/>
-      <xacro:default_transmission number="4"/>
-      <!-- <rgb camera> -->
-      <link name="rgb_camera">
-        <xacro:default_inertial mass="0.01"/>
-         <visual>
-             <origin rpy="-1.57 0 -1.57" xyz="-0.1 0.125 0.15"/>
-             <geometry>
-                 <mesh filename="package://hannahbot_description/meshes/pi_camera.STL" scale="0.01 0.01 0.01"/>
-             </geometry>
-          </visual>
-          <collision>
-             <origin rpy="-1.57 0 -1.57" xyz="-0.1 0.125 0.15"/>
-             <geometry>
-                 <mesh filename="package://hannahbot_description/meshes/pi_camera.STL" scale="0.01 0.01 0.01"/>
-             </geometry>
-          </collision>
-      </link>
-      <joint name ="rgb_camera_joint" type="fixed">
-        <parent link="base_link"/>
-        <child link = "rgb_camera"/>
-        <origin xyz="0 0.45 0.2" rpy="0 -0.5 1.57"/>
     </joint>
-    <gazebo reference="rgb_camera">
-        <sensor type="camera" name="rgb_camera">
-            <always_on>true</always_on>
-            <update_rate>30.0</update_rate>
-            <camera name="rgb_camera">
-                <horizontal_fov>1.15</horizontal_fov>
-                <vertical_fov>0.71</vertical_fov>
-                <image>
-                    <width>2304</width>
-                    <height>1296</height>
-                    <format>R8G8B8</format>
-                </image>
-                <distortion>
-                    <k1>0.0</k1>
-                    <k2>0.0</k2>
-                    <k3>0.0</k3>
-                    <p1>0.0</p1>
-                    <p2>0.0</p2>
-                    <center>0.5 0.5</center>
-                </distortion>
-            </camera>
-            <plugin name="plugin_name" filename="libgazebo_ros_camera.so">
-                <ros>
-                    <remapping>~/image_raw:=image_raw</remapping>
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
File: hannahbot_description/urdf/hannahbot_gazebo.xacro (robot description, xacro)
@@ -1,10 +1,18 @@
 <?xml version="1.0"?>
-<robot xmlns:xacro="http://www.ros.org/wiki/xacro" name="hannah_bot">
-    <gazebo>
-        <plugin filename="libgazebo_ros2_control.so" name="gazebo_ros2_control">
-            <robot_param>robot_description</robot_param>
-            <robot_param_node>robot_state_publisher</robot_param_node>
-            <parameters>$(find hannahbot_controller)/config/hannah_controllers.yaml</parameters>
-        </plugin>
-    </gazebo>
+<robot xmlns:xacro="http://www.ros.org/wiki/xacro" name="hannahbot">
+  <!-- ROS 2 Control -->
+  <gazebo>
+    <!-- ROS 2 Humble -->
+    <xacro:if value="$(arg is_ignition)">
+      <plugin filename="ign_ros2_control-system" name="ign_ros2_control::IgnitionROS2ControlPlugin">
+        <parameters>$(find hannahbot_controller)/config/hannah_controllers.yaml</parameters>
+      </plugin>
+    </xacro:if>
+    <!-- ROS 2 Iron or above -->
+    <xacro:unless value="$(arg is_ignition)">
+      <plugin filename="gz_ros2_control-system" name="gz_ros2_control::GazeboSimROS2ControlPlugin">
+        <parameters>$(find hannahbot_controller)/config/hannah_controllers.yaml</parameters>
+      </plugin>
+    </xacro:unless>
+  </gazebo>
 </robot>

File: hannahbot_description/urdf/hannahbot_ros2_control.xacro (robot description, xacro)
@@ -1,21 +1,30 @@
 <?xml version="1.0"?>
-<robot xmlns:xacro="http://www.ros.org/wiki/xacro" name="hannah_bot">
-    <xacro:property name="PI" value="3.14159"/>
+<robot xmlns:xacro="http://www.ros.org/wiki/xacro" name="hannahbot">
     <ros2_control name="RobotSystem" type="system">
-        <hardware>
-            <plugin>gazebo_ros2_control/GazeboSystem</plugin>
-        </hardware>
+        <xacro:property name="PI" value="3.14159265359" />
+        <!-- ros2_control Gazebo -->
+        <!-- ROS 2 Humble -->
+        <xacro:if value="$(arg is_ignition)">
+            <hardware>
+                <plugin>ign_ros2_control/IgnitionSystem</plugin>
+            </hardware>
+        </xacro:if>
+        <!-- ROS 2 Iron or above -->
+        <xacro:unless value="$(arg is_ignition)">
+            <hardware>
+                <plugin>gz_ros2_control/GazeboSimSystem</plugin>
+            </hardware>
+        </xacro:unless>
         <joint name="joint_1">
-            <command_interface name="position">   <!-- used to send commands to the bot  -->
-                <param name="min">-${PI/2}</param>
-                <param name="max">${PI/2}</param>
+            <command_interface name="position">
+            <param name="min">-${PI / 2}</param>
+            <param name="max">${PI / 2}</param>
             </command_interface>
-            <!-- used to read the state of the robot -->
             <state_interface name="position"/>
         </joint>
         <joint name="joint_2">
             <command_interface name="position">
-                <param name="min">-${PI/2}</param>
-                <param name="max">${PI/2}</param>
+            <param name="min">-${PI / 2}</param>
+            <param name="max">${PI / 2}</param>
             </command_interface>
             <state_interface name="position"/>
@@ -23,13 +32,6 @@
         <joint name="joint_3">
             <command_interface name="position">
-                <param name="min">-${PI/2}</param>
-                <param name="max">${PI/2}</param>
-            </command_interface>
-            <state_interface name="position"/>
-        </joint>
-        <joint name="hori_arm_claw_joint">
-            <command_interface name="position">
-                <param name="min">-${PI/2}</param>
-                <param name="max">${PI/2}</param>
+            <param name="min">-${PI / 2}</param>
+            <param name="max">${PI / 2}</param>
             </command_interface>
             <state_interface name="position"/>
@@ -37,18 +39,12 @@
         <joint name="joint_4">
             <command_interface name="position">
-                <param name="min">-${PI/2}</param>
-                <param name="max">0.0</param>
+            <param name="min">-${PI / 2}</param>
+            <param name="max">0.0</param>
             </command_interface>
             <state_interface name="position"/>
         </joint>
         <joint name="joint_5">
-        <!-- These parameters in the joint_5 states that the its gonna mimic joint_4 and the -1 means in the opposite direction -->
             <param name="mimic">joint_4</param>
             <param name="multiplier">-1</param>
-            <command_interface name="position">
-                <param name="min">0.0</param>
-                <param name="max">${PI/2}</param>
-            </command_interface>
-            <state_interface name="position"/>
         </joint>
     </ros2_control>
